File: src/CMOS-Clock-V1.kicad_pcb (KiCad board)
At the start: 4 copper layers, 100 x 61 mm, 102 parts, among them J1 USB_B_Micro, SW1 SW_Push, SW2 SW_Push, SW3 SW_Push, U1 BAS28,215, U10 74AHC86D,118, U11 74HC390D,652, U12 74HC390D,652, U13 2N7002PS, U14 MC14511BDR2G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

Commit message: Update
Other:
- net class Default removed
